Commit message: Update robot_core.xacro

File: description/robot_core.xacro (robot description, xacro)
@@ -2,5 +2,5 @@
 <robot xmlns:xacro="http://www.ros.org/wiki/xacro">
   <!-- Includes -->
-  <!-- <xacro:include filename="inertial_macros.xacro"/> -->
+  <xacro:include filename="inertial_macros.xacro"/>
   <!-- Materials -->
   <material name="silver">
@@ -8,8 +8,17 @@
   </material>
   <!-- World and Base Reference -->
+  <link name="universe">
+  <!-- Probably edit world joint origin to move gripper start position arround-->
+  <joint name="world_joint" type="fixed">
+    <parent link="universe"/>
+    <child link="world"/>
+    <origin xyz="0 0 0" rpy="0 0 0"/>
+  </joint>
   <link name="world"/>
-  <joint name="world_joint" type="fixed">
-    <parent link="world"/>
+  </link>
+  <joint name="base_link_joint" type="fixed">
+    <parent link="universe"/>
     <child link="base_link"/>
+    <origin xyz="0 0 0" rpy="0 0 0"/>
   </joint>
   <!-- Link Definitions -->

Commit message: putting inertial last in links, making all link structures equal

File: description/robot_core.xacro (robot description, xacro)
@@ -52,4 +52,17 @@
   </link>
   <link name="Component5_1">
+    <visual>
+      <origin xyz="0.011816 -0.035888 -0.012432" rpy="0 0 0"/>
+      <geometry>
+        <mesh filename="file://$(find gripperbot)/meshes/Component5_1.stl" scale="0.001 0.001 0.001"/>
+      </geometry>
+      <material name="silver"/>
+    </visual>
+    <collision>
+      <origin xyz="0.011816 -0.035888 -0.012432" rpy="0 0 0"/>
+      <geometry>
+        <mesh filename="file://$(find gripperbot)/meshes/Component5_1.stl" scale="0.001 0.001 0.001"/>
+      </geometry>
+    </collision>
     <inertial>
       <origin xyz="-2.8632491516460135e-07 -4.6737513356405816e-07 -0.04667345672442119" rpy="0 0 0"/>
@@ -57,19 +70,19 @@
       <inertia ixx="0.002572" ixy="0.000177" ixz="0" iyy="0.002954" iyz="0" izz="0.002679"/>
     </inertial>
-    <visual>
-      <origin xyz="0.011816 -0.035888 -0.012432" rpy="0 0 0"/>
-      <geometry>
-        <mesh filename="file://$(find gripperbot)/meshes/Component5_1.stl" scale="0.001 0.001 0.001"/>
-      </geometry>
-      <material name="silver"/>
-    </visual>
-    <collision>
-      <origin xyz="0.011816 -0.035888 -0.012432" rpy="0 0 0"/>
-      <geometry>
-        <mesh filename="file://$(find gripperbot)/meshes/Component5_1.stl" scale="0.001 0.001 0.001"/>
-      </geometry>
-    </collision>
   </link>
   <link name="Component1_1">
+    <visual>
+      <origin xyz="-0.048184 -0.035888 -0.137432" rpy="0 0 0"/>
+      <geometry>
+        <mesh filename="file://$(find gripperbot)/meshes/Component1_1.stl" scale="0.001 0.001 0.001"/>
+      </geometry>
+      <material name="silver"/>
+    </visual>
+    <collision>
+      <origin xyz="-0.048184 -0.035888 -0.137432" rpy="0 0 0"/>
+      <geometry>
+        <mesh filename="file://$(find gripperbot)/meshes/Component1_1.stl" scale="0.001 0.001 0.001"/>
+      </geometry>
+    </collision>
     <inertial>
       <origin xyz="-0.06000028632491587 -4.6737513197765354e-07 -0.007836367251077725" rpy="0 0 0"/>
@@ -77,19 +90,19 @@
       <inertia ixx="0.002538" ixy="0" ixz="0" iyy="0.004372" iyz="0" izz="0.005986"/>
     </inertial>
-    <visual>
-      <origin xyz="-0.048184 -0.035888 -0.137432" rpy="0 0 0"/>
-      <geometry>
-        <mesh filename="file://$(find gripperbot)/meshes/Component1_1.stl" scale="0.001 0.001 0.001"/>
-      </geometry>
-      <material name="silver"/>
-    </visual>
-    <collision>
-      <origin xyz="-0.048184 -0.035888 -0.137432" rpy="0 0 0"/>
-      <geometry>
-        <mesh filename="file://$(find gripperbot)/meshes/Component1_1.stl" scale="0.001 0.001 0.001"/>
-      </geometry>
-    </collision>
   </link>
   <link name="Component3_1">
+    <visual>
+      <origin xyz="0.011816 -0.093388 -0.145432" rpy="0 0 0"/>
+      <geometry>
+        <mesh filename="file://$(find gripperbot)/meshes/Component3_1.stl" scale="0.001 0.001 0.001"/>
+      </geometry>
+      <material name="silver"/>
+    </visual>
+    <collision>
+      <origin xyz="0.011816 -0.093388 -0.145432" rpy="0 0 0"/>
+      <geometry>
+        <mesh filename="file://$(find gripperbot)/meshes/Component3_1.stl" scale="0.001 0.001 0.001"/>
+      </geometry>
+    </collision>
     <inertial>
       <origin xyz="-2.8632491584634767e-07 -0.007500467375131714 0.014999759238118415" rpy="0 0 0"/>
@@ -97,19 +110,19 @@
       <inertia ixx="3e-05" ixy="0" ixz="0" iyy="0.000238" iyz="0" izz="0.000221"/>
     </inertial>
-    <visual>
-      <origin xyz="0.011816 -0.093388 -0.145432" rpy="0 0 0"/>
-      <geometry>
-        <mesh filename="file://$(find gripperbot)/meshes/Component3_1.stl" scale="0.001 0.001 0.001"/>
-      </geometry>
-      <material name="silver"/>
-    </visual>
-    <collision>
-      <origin xyz="0.011816 -0.093388 -0.145432" rpy="0 0 0"/>
-      <geometry>
-        <mesh filename="file://$(find gripperbot)/meshes/Component3_1.stl" scale="0.001 0.001 0.001"/>
-      </geometry>
-    </collision>
   </link>
   <link name="Component9_1">
+    <visual>
+      <origin xyz="0.011816 0.021612 -0.145432" rpy="0 0 0"/>
+      <geometry>
+        <mesh filename="file://$(find gripperbot)/meshes/Component9_1.stl" scale="0.001 0.001 0.001"/>
+      </geometry>
+      <material name="silver"/>
+    </visual>
+    <collision>
+      <origin xyz="0.011816 0.021612 -0.145432" rpy="0 0 0"/>
+      <geometry>
+        <mesh filename="file://$(find gripperbot)/meshes/Component9_1.stl" scale="0.001 0.001 0.001"/>
+      </geometry>
+    </collision>
     <inertial>
       <origin xyz="-2.8632491608053534e-07 0.0074995326248675845 0.014999759238119414" rpy="0 0 0"/>
@@ -117,19 +130,19 @@
       <inertia ixx="3e-05" ixy="0" ixz="0" iyy="0.000238" iyz="0" izz="0.000221"/>
     </inertial>
-    <visual>
-      <origin xyz="0.011816 0.021612 -0.145432" rpy="0 0 0"/>
-      <geometry>
-        <mesh filename="file://$(find gripperbot)/meshes/Component9_1.stl" scale="0.001 0.001 0.001"/>
-      </geometry>
-      <material name="silver"/>
-    </visual>
-    <collision>
-      <origin xyz="0.011816 0.021612 -0.145432" rpy="0 0 0"/>
-      <geometry>
-        <mesh filename="file://$(find gripperbot)/meshes/Component9_1.stl" scale="0.001 0.001 0.001"/>
-      </geometry>
-    </collision>
   </link>
   <link name="Component10_1">
+    <visual>
+      <origin xyz="0.009964 0.00974 0.030135" rpy="0 0 0"/>
+      <geometry>
+        <mesh filename="file://$(find gripperbot)/meshes/Component10_1.stl" scale="0.001 0.001 0.001"/>
+      </geometry>
+      <material name="silver"/>
+    </visual>
+    <collision>
+      <origin xyz="0.009964 0.00974 0.030135" rpy="0 0 0"/>
+      <geometry>
+        <mesh filename="file://$(find gripperbot)/meshes/Component10_1.stl" scale="0.001 0.001 0.001"/>
+      </geometry>
+    </collision>
     <inertial>
       <origin xyz="-0.006984004938344654 0.002734264130490712 -0.015000240761882375" rpy="0 0 0"/>
@@ -137,19 +150,19 @@
       <inertia ixx="0.000211" ixy="-7.1e-05" ixz="0" iyy="5.8e-05" iyz="0" izz="0.000221"/>
     </inertial>
-    <visual>
-      <origin xyz="0.009964 0.00974 0.030135" rpy="0 0 0"/>
-      <geometry>
-        <mesh filename="file://$(find gripperbot)/meshes/Component10_1.stl" scale="0.001 0.001 0.001"/>
-      </geometry>
-      <material name="silver"/>
-    </visual>
-    <collision>
-      <origin xyz="0.009964 0.00974 0.030135" rpy="0 0 0"/>
-      <geometry>
-        <mesh filename="file://$(find gripperbot)/meshes/Component10_1.stl" scale="0.001 0.001 0.001"/>
-      </geometry>
-    </collision>
   </link>
   <link name="Component8_1">
+    <visual>
+      <origin xyz="0.066074 -0.054923 0.062568" rpy="0 0 0"/>
+      <geometry>
+        <mesh filename="file://$(find gripperbot)/meshes/Component8_1.stl" scale="0.001 0.001 0.001"/>
+      </geometry>
+      <material name="silver"/>
+    </visual>
+    <collision>
+      <origin xyz="0.066074 -0.054923 0.062568" rpy="0 0 0"/>
+      <geometry>
+        <mesh filename="file://$(find gripperbot)/meshes/Component8_1.stl" scale="0.001 0.001 0.001"/>
+      </geometry>
+    </collision>
     <inertial>
       <origin xyz="0.006983432288514446 -0.0027341988807576927 -0.015000240761882014" rpy="0 0 0"/>
@@ -157,17 +170,4 @@
       <inertia ixx="0.000211" ixy="-7.1e-05" ixz="0" iyy="5.8e-05" iyz="0" izz="0.000221"/>
     </inertial>
-    <visual>
-      <origin xyz="0.066074 -0.054923 0.062568" rpy="0 0 0"/>
-      <geometry>
-        <mesh filename="file://$(find gripperbot)/meshes/Component8_1.stl" scale="0.001 0.001 0.001"/>
-      </geometry>
-      <material name="silver"/>
-    </visual>
-    <collision>
-      <origin xyz="0.066074 -0.054923 0.062568" rpy="0 0 0"/>
-      <geometry>
-        <mesh filename="file://$(find gripperbot)/meshes/Component8_1.stl" scale="0.001 0.001 0.001"/>
-      </geometry>
-    </collision>
   </link>
   <!-- Joint Definitions -->
